Commit message: update

File: description/robot_core.xacro (robot description, xacro)
@@ -1,5 +1,5 @@
 <?xml version="1.0"?>
 <robot xmlns:xacro="http://www.ros.org/wiki/xacro">
-    <xacro include filename="inertial_macros.xacro"/>
+    <xacro:include filename="inertial_macros.xacro"/>
     <!-- Colours for use in URDF declared below:-->
     <material name="white">
@@ -41,20 +41,23 @@
     <link name="chassis_link">
         <visual>
-        <origin xyz="0.125 0 -0.025"/>
-        <geometry>
-            <box size= "0.25 0.16 0.05"/>
-        </geometry>
-        <material name="black"/>
+            <origin xyz="0.125 0 -0.025"/>
+            <geometry>
+                <box size= "0.25 0.16 0.05"/>
+            </geometry>
+            <material name="black"/>
         </visual>
         <collision>
-        <origin xyz="0.125 0 -0.025"/>
-        <geometry>
-            <box size= "0.25 0.16 0.05"/>
-        </geometry>
+            <origin xyz="0.125 0 -0.025"/>
+            <geometry>
+                <box size= "0.25 0.16 0.05"/>
+            </geometry>
         </collision>
-        <xacro:inetrial_box mass="0.5" x="0.25" y="0.16" z="0.05">
+        <xacro:inertial_box mass="0.5" x="0.25" y="0.16" z="0.05">
             <origin xyz="0.125 0 -0.025" rpy="0 0 0"/>
         </xacro:inertial_box>
     </link>
+    <gazebo reference="chassis_link">
+        <material>Gazebo/Black</material>
+    </gazebo>
     <!-- Wheel Links: -->
     <!-- Left Wheel Links: -->
@@ -68,20 +71,23 @@
     <link name="left_wheel_rear_link">
         <visual>
-        <origin xyz="0 0 0.01425"/>
+            <origin xyz="0 0 0.01425"/>
             <geometry>
-                <cylinder radius="0.033" length="0.0285"/>
+                <cylinder radius="0.035" length="0.0285"/>
             </geometry>
             <material name="yellow"/>
         </visual>
         <collision>
-        <origin xyz="0 0 0.01425"/>
+            <origin xyz="0 0 0.01425"/>
             <geometry>
-                <cylinder radius="0.033" length="0.0285"/>
+                <cylinder radius="0.035" length="0.0285"/>
             </geometry>
         </collision>
-        <xacro:inertial_cylinder mass="0.1" radius="0.033" length="0.0285">
+        <xacro:inertial_cylinder mass="0.1" radius="0.035" length="0.0285">
             <origin xyz="0 0 0.01425" rpy="0 0 0"/>
-        <xacro:inertial_cylinder/>
+        </xacro:inertial_cylinder>
     </link>
+    <gazebo reference="left_wheel_rear_link">
+        <material>Gazebo/Yellow</material>
+    </gazebo>
     <!-- FWD -->
     <joint name="left_wheel_fwd_joint" type="continuous">
@@ -93,21 +99,24 @@
     <link name="left_wheel_fwd_link">
         <visual>
-        <origin xyz="0 0 0.01425"/>
+            <origin xyz="0 0 0.01425"/>
             <geometry>
-                <cylinder radius="0.033" length="0.0285"/>
+                <cylinder radius="0.035" length="0.0285"/>
             </geometry>
             <material name="yellow"/>
         </visual>
         <collision>
-        <origin xyz="0 0 0.01425"/>
+            <origin xyz="0 0 0.01425"/>
             <geometry>
-                <cylinder radius="0.033" length="0.0285"/>
+                <cylinder radius="0.035" length="0.0285"/>
             </geometry>
         </collision>
-        <xacro:inertial_cylinder mass="0.1" radius="0.033" length="0.0285">
+        <xacro:inertial_cylinder mass="0.1" radius="0.035" length="0.0285">
             <origin xyz="0 0 0.01425" rpy="0 0 0"/>
-        <xacro:inertial_cylinder/>
+        </xacro:inertial_cylinder>
     </link>
-        <!-- Right Wheel Links: -->
+    <gazebo reference="left_wheel_fwd_link">
+        <material>Gazebo/Yellow</material>
+    </gazebo>
+    <!-- Right Wheel Links: -->
     <!-- REAR -->
     <joint name="right_wheel_rear_joint" type="continuous">
@@ -119,20 +128,23 @@
     <link name="right_wheel_rear_link">
         <visual>
-        <origin xyz="0 0 0.01425"/>
+            <origin xyz="0 0 0.01425"/>
             <geometry>
-                <cylinder radius="0.033" length="0.0285"/>
+                <cylinder radius="0.035" length="0.0285"/>
             </geometry>
             <material name="yellow"/>
         </visual>
         <collision>
-        <origin xyz="0 0 0.01425"/>
+            <origin xyz="0 0 0.01425"/>
             <geometry>
-                <cylinder radius="0.033" length="0.0285"/>
+                <cylinder radius="0.035" length="0.0285"/>
             </geometry>
         </collision>
-        <xacro:inertial_cylinder mass="0.1" radius="0.033" length="0.0285">
+        <xacro:inertial_cylinder mass="0.1" radius="0.035" length="0.0285">
             <origin xyz="0 0 0.01425" rpy="0 0 0"/>
-        <xacro:inertial_cylinder/>
+        </xacro:inertial_cylinder>
     </link>
+    <gazebo reference="right_wheel_rear_link">
+        <material>Gazebo/Yellow</material>
+    </gazebo>
     <!-- FWD -->
     <joint name="right_wheel_fwd_joint" type="continuous">
@@ -144,19 +156,22 @@
     <link name="right_wheel_fwd_link">
         <visual>
-        <origin xyz="0 0 0.01425"/>
+            <origin xyz="0 0 0.01425"/>
             <geometry>
-                <cylinder radius="0.033" length="0.0285"/>
+                <cylinder radius="0.035" length="0.0285"/>
             </geometry>
             <material name="yellow"/>
         </visual>
         <collision>
-        <origin xyz="0 0 0.01425"/>
+            <origin xyz="0 0 0.01425"/>
             <geometry>
-                <cylinder radius="0.033" length="0.0285"/>
+                <cylinder radius="0.035" length="0.0285"/>
             </geometry>
         </collision>
-        <xacro:inertial_cylinder mass="0.1" radius="0.033" length="0.0285">
+        <xacro:inertial_cylinder mass="0.1" radius="0.035" length="0.0285">
             <origin xyz="0 0 0.01425" rpy="0 0 0"/>
-        <xacro:inertial_cylinder/>
+        </xacro:inertial_cylinder>
     </link>
+    <gazebo reference="right_wheel_fwd_link">
+        <material>Gazebo/Yellow</material>
+    </gazebo>
 </robot>
