Commit message: cam_node launch, xacro files

File: description/lidar.xacro (robot description, xacro)
@@ -25,4 +25,5 @@
     </link>
     <gazebo reference="laser_frame">
+     <material>Gazebo/Grey</material>
         <sensor name="laser" type="ray">
             <pose>0 0 0 0 0 0</pose>

File: description/robot.urdf.xacro (robot description, xacro)
@@ -4,3 +4,4 @@
     <xacro:include filename="gazebo_control.xacro"/>
     <xacro:include filename="lidar.xacro"/>
+    <xacro:include filename="camera.xacro"/>
 </robot>
