Commit message: updated description

File: description/gazebo_control.xacro (robot description, xacro)
@@ -1,4 +1,4 @@
 <?xml version="1.0"?>
-<robot name="my_robot" xmlns:xacro="http://www.ros.org/wiki/xacro">
+<robot xmlns:xacro="http://www.ros.org/wiki/xacro">
     <!-- Gazebo Plugin for Diff Drive -->
     <gazebo>
@@ -14,5 +14,5 @@
             <wheel_diameter>0.07</wheel_diameter>       <!-- Diameter of the wheels -->
             <!-- Drive parameters -->
-            <max_wheel_torque>200</max_wheel_torque>
+            <max_wheel_torque>100</max_wheel_torque>
             <max_wheel_acceleration>10.0</max_wheel_acceleration>
             <!-- Frames -->

File: description/lidar.xacro (robot description, xacro)
@@ -8,5 +8,5 @@
     <link name="laser_frame">
         <visual>
-            <origin xyz="0 0 0" rpy="0 0 0"/>
+            <origin xyz="0 0 0.03" rpy="0 0 0"/>
             <geometry>
                 <cylinder length="0.04" radius="0.055"/>
@@ -27,5 +27,5 @@
      <material>Gazebo/Grey</material>
         <sensor name="laser" type="ray">
-            <pose>0 0 0 0 0 0</pose>
+            <pose>0 0 0.035 0 0 0</pose>
             <visualize>true</visualize>
             <update_rate>10</update_rate>

File: description/robot.urdf.xacro (robot description, xacro)
@@ -1,7 +1,6 @@
 <?xml version="1.0"?>
-<robot xmlns:xacro="http://www.ros.org/wiki/xacro" name="robot">
+<robot xmlns:xacro="http://www.ros.org/wiki/xacro"  name="robot">
     <xacro:include filename="robot_core.xacro"/>
     <xacro:include filename="gazebo_control.xacro"/>
     <xacro:include filename="lidar.xacro"/>
-    <xacro:include filename="camera.xacro"/>
 </robot>

File: description/robot_core.xacro (robot description, xacro)
@@ -43,5 +43,5 @@
             <origin xyz="0.125 0 -0.025"/>
             <geometry>
-                <box size= "0.25 0.16 0.05"/>
+                <box size= "0.30 0.20 0.05"/>
             </geometry>
             <material name="black"/>
@@ -50,8 +50,8 @@
             <origin xyz="0.125 0 -0.025"/>
             <geometry>
-                <box size= "0.25 0.16 0.05"/>
+                <box size= "0.30 0.20 0.05"/>
             </geometry>
         </collision>
-        <xacro:inertial_box mass="0.5" x="0.25" y="0.16" z="0.05">
+        <xacro:inertial_box mass="0.5" x="0.30" y="0.20" z="0.05">
             <origin xyz="0.125 0 -0.025" rpy="0 0 0"/>
         </xacro:inertial_box>
@@ -66,5 +66,5 @@
         <parent link="base_link"/>
         <child link="left_wheel_rear_link"/>
-        <origin xyz="-0.0635 0.08 0" rpy="-${pi/2} 0 0"/>
+        <origin xyz="-0.125 0.10 0" rpy="-${pi/2} 0 0"/>
         <axis xyz="0 0 1"/>
     </joint>
@@ -73,20 +73,20 @@
             <origin xyz="0 0 0.01425"/>
             <geometry>
-                <cylinder radius="0.035" length="0.0285"/>
+                <cylinder radius="0.05" length="0.04"/>
             </geometry>
-            <material name="yellow"/>
+            <material name="grey"/>
         </visual>
         <collision>
             <origin xyz="0 0 0.01425"/>
             <geometry>
-                <cylinder radius="0.035" length="0.0285"/>
+                <cylinder radius="0.05" length="0.04"/>
             </geometry>
         </collision>
-        <xacro:inertial_cylinder mass="0.1" radius="0.035" length="0.0285">
+        <xacro:inertial_cylinder mass="0.1" radius="0.05" length="0.04">
             <origin xyz="0 0 0.01425" rpy="0 0 0"/>
         </xacro:inertial_cylinder>
     </link>
     <gazebo reference="left_wheel_rear_link">
-        <material>Gazebo/Yellow</material>
+        <material>Gazebo/Grey</material>
     </gazebo>
     <!-- FWD -->
@@ -94,5 +94,5 @@
         <parent link="base_link"/>
         <child link="left_wheel_fwd_link"/>
-        <origin xyz="0.0635 0.08 0" rpy="-${pi/2} 0 0"/>
+        <origin xyz="0.125 0.10 0" rpy="-${pi/2} 0 0"/>
         <axis xyz="0 0 1"/>
     </joint>
@@ -101,20 +101,20 @@
             <origin xyz="0 0 0.01425"/>
             <geometry>
-                <cylinder radius="0.035" length="0.0285"/>
+                <cylinder radius="0.05" length="0.04"/>
             </geometry>
-            <material name="yellow"/>
+            <material name="grey"/>
         </visual>
         <collision>
             <origin xyz="0 0 0.01425"/>
             <geometry>
-                <cylinder radius="0.035" length="0.0285"/>
+                <cylinder radius="0.05" length="0.04"/>
             </geometry>
         </collision>
-        <xacro:inertial_cylinder mass="0.1" radius="0.035" length="0.0285">
+        <xacro:inertial_cylinder mass="0.1" radius="0.05" length="0.04">
             <origin xyz="0 0 0.01425" rpy="0 0 0"/>
         </xacro:inertial_cylinder>
     </link>
     <gazebo reference="left_wheel_fwd_link">
-        <material>Gazebo/Yellow</material>
+        <material>Gazebo/Grey</material>
     </gazebo>
     <!-- Right Wheel Links: -->
@@ -123,5 +123,5 @@
         <parent link="base_link"/>
         <child link="right_wheel_rear_link"/>
-        <origin xyz="-0.0635 -0.08 0" rpy="${pi/2} 0 0"/>
+        <origin xyz="-0.125 -0.10 0" rpy="${pi/2} 0 0"/>
         <axis xyz="0 0 -1"/>
     </joint>
@@ -130,20 +130,20 @@
             <origin xyz="0 0 0.01425"/>
             <geometry>
-                <cylinder radius="0.035" length="0.0285"/>
+                <cylinder radius="0.05" length="0.04"/>
             </geometry>
-            <material name="yellow"/>
+            <material name="grey"/>
         </visual>
         <collision>
             <origin xyz="0 0 0.01425"/>
             <geometry>
-                <cylinder radius="0.035" length="0.0285"/>
+                <cylinder radius="0.05" length="0.04"/>
             </geometry>
         </collision>
-        <xacro:inertial_cylinder mass="0.1" radius="0.035" length="0.0285">
+        <xacro:inertial_cylinder mass="0.1" radius="0.05" length="0.04">
             <origin xyz="0 0 0.01425" rpy="0 0 0"/>
         </xacro:inertial_cylinder>
     </link>
     <gazebo reference="right_wheel_rear_link">
-        <material>Gazebo/Yellow</material>
+        <material>Gazebo/Grey</material>
     </gazebo>
     <!-- FWD -->
@@ -151,5 +151,5 @@
         <parent link="base_link"/>
         <child link="right_wheel_fwd_link"/>
-        <origin xyz="0.0635 -0.08 0" rpy="${pi/2} 0 0"/>
+        <origin xyz="0.125 -0.10 0" rpy="${pi/2} 0 0"/>
         <axis xyz="0 0 -1"/>
     </joint>
@@ -158,20 +158,20 @@
             <origin xyz="0 0 0.01425"/>
             <geometry>
-                <cylinder radius="0.035" length="0.0285"/>
+                <cylinder radius="0.05" length="0.04"/>
             </geometry>
-            <material name="yellow"/>
+            <material name="grey"/>
         </visual>
         <collision>
             <origin xyz="0 0 0.01425"/>
             <geometry>
-                <cylinder radius="0.035" length="0.0285"/>
+                <cylinder radius="0.05" length="0.04"/>
             </geometry>
         </collision>
-        <xacro:inertial_cylinder mass="0.1" radius="0.035" length="0.0285">
+        <xacro:inertial_cylinder mass="0.1" radius="0.05" length="0.04">
             <origin xyz="0 0 0.01425" rpy="0 0 0"/>
         </xacro:inertial_cylinder>
     </link>
     <gazebo reference="right_wheel_fwd_link">
-        <material>Gazebo/Yellow</material>
+        <material>Gazebo/Grey</material>
     </gazebo>
 </robot>

Commit message: Config changes and Robot Launch File

File: description/gazebo_control.xacro (robot description, xacro)
@@ -11,6 +11,6 @@
             <right_joint>right_wheel_fwd_joint</right_joint>
             <!-- Wheel parameters -->
-            <wheel_separation>0.16</wheel_separation>  <!-- Distance between left and right wheels -->
-            <wheel_diameter>0.07</wheel_diameter>       <!-- Diameter of the wheels -->
+            <wheel_separation>0.20</wheel_separation>  <!-- Distance between left and right wheels -->
+            <wheel_diameter>0.10</wheel_diameter>       <!-- Diameter of the wheels -->
             <!-- Drive parameters -->
             <max_wheel_torque>100</max_wheel_torque>

File: description/robot.urdf.xacro (robot description, xacro)
@@ -2,5 +2,6 @@
 <robot xmlns:xacro="http://www.ros.org/wiki/xacro"  name="robot">
     <xacro:include filename="robot_core.xacro"/>
-    <xacro:include filename="gazebo_control.xacro"/>
+   <!-- <xacro:include filename="gazebo_control.xacro"/> -->
+    <xacro:include filename="ros2_control.xacro"/>
     <xacro:include filename="lidar.xacro"/>
 </robot>

File: description/robot_core.xacro (robot description, xacro)
@@ -66,5 +66,5 @@
         <parent link="base_link"/>
         <child link="left_wheel_rear_link"/>
-        <origin xyz="-0.125 0.10 0" rpy="-${pi/2} 0 0"/>
+        <origin xyz="-0.125 0.106 0" rpy="-${pi/2} 0 0"/>
         <axis xyz="0 0 1"/>
     </joint>
@@ -80,5 +80,5 @@
             <origin xyz="0 0 0.01425"/>
             <geometry>
-                <cylinder radius="0.05" length="0.04"/>
+                <sphere radius="0.05" />
             </geometry>
         </collision>
@@ -94,5 +94,5 @@
         <parent link="base_link"/>
         <child link="left_wheel_fwd_link"/>
-        <origin xyz="0.125 0.10 0" rpy="-${pi/2} 0 0"/>
+        <origin xyz="0.125 0.106 0" rpy="-${pi/2} 0 0"/>
         <axis xyz="0 0 1"/>
     </joint>
@@ -108,5 +108,5 @@
             <origin xyz="0 0 0.01425"/>
             <geometry>
-                <cylinder radius="0.05" length="0.04"/>
+                <sphere radius="0.05"/>
             </geometry>
         </collision>
@@ -123,5 +123,5 @@
         <parent link="base_link"/>
         <child link="right_wheel_rear_link"/>
-        <origin xyz="-0.125 -0.10 0" rpy="${pi/2} 0 0"/>
+        <origin xyz="-0.125 -0.106 0" rpy="${pi/2} 0 0"/>
         <axis xyz="0 0 -1"/>
     </joint>
@@ -137,5 +137,5 @@
             <origin xyz="0 0 0.01425"/>
             <geometry>
-                <cylinder radius="0.05" length="0.04"/>
+                <sphere radius="0.05"/>
             </geometry>
         </collision>
@@ -151,5 +151,5 @@
         <parent link="base_link"/>
         <child link="right_wheel_fwd_link"/>
-        <origin xyz="0.125 -0.10 0" rpy="${pi/2} 0 0"/>
+        <origin xyz="0.125 -0.106 0" rpy="${pi/2} 0 0"/>
         <axis xyz="0 0 -1"/>
     </joint>
@@ -165,5 +165,5 @@
             <origin xyz="0 0 0.01425"/>
             <geometry>
-                <cylinder radius="0.05" length="0.04"/>
+                <sphere radius="0.05"/>
             </geometry>
         </collision>
